Commit message: feat(hardware): integrate ros2_control Gazebo plugins and unmock MoveIt C++ execution node

File: src/vla_description/urdf/vla_arm.urdf.xacro (robot description, xacro)
@@ -90,3 +90,30 @@
     <origin xyz="0 0 0.4" rpy="0 0 0"/>
   </joint>
+  <!-- ros2_control integration for Gazebo -->
+  <ros2_control name="GazeboSimSystem" type="system">
+    <hardware>
+      <plugin>gz_ros2_control/GazeboSimSystem</plugin>
+    </hardware>
+    <joint name="joint_1">
+      <command_interface name="position">
+        <param name="min">-3.14</param>
+        <param name="max">3.14</param>
+      </command_interface>
+      <state_interface name="position"/>
+      <state_interface name="velocity"/>
+    </joint>
+    <joint name="joint_2">
+      <command_interface name="position">
+        <param name="min">-1.57</param>
+        <param name="max">1.57</param>
+      </command_interface>
+      <state_interface name="position"/>
+      <state_interface name="velocity"/>
+    </joint>
+  </ros2_control>
+  <gazebo>
+    <plugin filename="gz_ros2_control-system" name="gz_ros2_control::GazeboSimSystem">
+      <parameters>$(find vla_description)/config/ros2_controllers.yaml</parameters>
+    </plugin>
+  </gazebo>
 </robot>
